File: PCB Files/ENGR357_Project_v1.1.kicad_pcb (KiCad board)
At the start: 2 copper layers, 100 x 100 mm, 80 parts, among them J1 Conn_01x02_Female, J10 IQ_SDR-rescue_Conn_01x01-Conn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, J11 IQ_SDR-rescue_Conn_01x01-Conn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, J12 IQ_SDR-rescue_Conn_01x01-Conn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, J13 IQ_SDR-rescue_Conn_01x01-Conn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, J14 IQ_SDR-rescue_Conn_01x01-Conn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, J15 IQ_SDR-rescue_Conn_01x01-Conn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, J16 IQ_SDR-rescue_Conn_01x01-Conn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, J17 IQ_SDR-rescue_Conn_01x01-Conn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, J2 Conn_01x02_Female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

Commit message: Add files via upload
Parts:
- moved J6 17.2 mm to (75.5, 80.0), turned to 0 degrees
- moved R1 9.34 mm to (90.0, 89.0), turned to 90 degrees
Routing:
- net Net-(C7-Pad2): track 12.5 -> 33.1 mm
- net +3V3: track 88.3 -> 79.5 mm
- net /SCL_3V: track 46.5 -> 53.2 mm
- net Net-(J6-Pad2): track 27.3 -> 30.7 mm
Other:
- board text added: "Bandpass Filter"
- board text added: "Crystal"
- board text added: "Instrumentation Amplifiers"
- board text added: "Low-Pass Filter"
- board text added: "Tayloe Mixer"
- board text added: "Voltage Smoother"
